Commit message: urdf modified

File: install/description/share/description/urdf/armybot.urdf.xacro (robot description, xacro)
@@ -1,267 +1,85 @@
-<?xml version="1.0" ?>
-  <robot name="rover">
-  <link name="chassis">
+<?xml version="1.0"?>
+<robot name="rover">
+  <link name="base_link">
+  <visual>
+    <geometry>
+      <box size="0 0 0"/>
+    </geometry>
+    <material name="red">
+      <color rgba="1 0 0 1"/>
+    </material>
+  </visual>
+</link>
+<link name="left_wheel">
+  <visual>
+    <geometry>
+      <cylinder radius="0.04" length="0.05" />
+    </geometry>
+    <material name="red">
+      <color rgba="1 0 0 1"/>
+    </material>
+  </visual>
+</link>
+<link name="right_wheel">
+  <visual>
+    <geometry>
+      <cylinder radius="0.04" length="0.05" />
+    </geometry>
+    <material name="red">
+      <color rgba="1 0 0 1"/>
+    </material>
+  </visual>
+</link>
+<joint name="base_link_left_wheel" type="continuous">
+  <axis xyz="0.0 0.0 1" />
+  <parent link="base_link" />
+  <child link="left_wheel" />
+  <origin xyz="1.5 0 0" rpy="-1.5 0 0" />
+</joint>
+<joint name="base_link_right_wheel" type="continuous">
+  <axis xyz="0.0 0.0 1" />
+  <parent link="base_link" />
+  <child link="right_wheel" />
+  <origin xyz="-1.5 0 0" rpy="-1.5 0 0" />
+</joint>
+<link name="left_wheel_backside">
     <visual>
       <geometry>
-          <box size=".8 0.7 0.1"/>
+        <cylinder radius="0.04" length="0.05" />
       </geometry>
-      <material name="gray">
-        <color rgba=".2 .2 .2 1" />
+      <material name="red">
+        <color rgba="1 0 0 1"/>
       </material>
     </visual>
-  <inertial>
-            <mass value="2" />
-            <inertia ixx="0.04" ixy="0.0" ixz="0"
-            iyy="0.17" iyz="0" izz="0.25" />
-    </inertial>
-    <collision>
-      <geometry>
-          <box size=".8 0.7 0.1"/>
-      </geometry>
-    </collision>
   </link>
-  <link name="wheel_front_right">
-    <inertial>
-            <mass value="2" />
-            <inertia ixx="1e-3" ixy="0.0" ixz="0"
-            iyy="1e-3" iyz="0" izz="1e-3" />
-    </inertial>
+  <joint name="base_link_left_wheel_backside" type="continuous">
+    <parent link="base_link" />
+    <child link="left_wheel_backside" />
+    <origin xyz="-0.2 0.2 -0.05" rpy="1.570796 0 0"/>
+  </joint>
+  <link name="right_wheel_frontside">
     <visual>
       <geometry>
-          <cylinder radius="0.15" length="0.1"/>
+        <cylinder radius="0.04" length="0.05" />
       </geometry>
-      <material name="white">
-        <color rgba="1 1 1 1"/>
+      <material name="red">
+        <color rgba="1 0 0 1"/>
       </material>
     </visual>
-    <collision>
-      <geometry>
-          <cylinder radius="0.15" length="0.1"/>
-      </geometry>
-      <contact_coefficients mu="1" kp="1e+13" kd="1.0"/>
-    </collision>
   </link>
-  <joint name="wheel_front_right_joint" type="continuous">
-    <origin xyz="0.25 0.4 0.0" rpy="1.57 0.0 0.0"/>
-    <parent link="chassis"/>
-    <child link="wheel_front_right"/>
-    <axis xyz="0.0 0.0 1.0"/>
+  <joint name="base_link_right_wheel_frontside" type="continuous">
+    <parent link="base_link" />
+    <child link="right_wheel_frontside" />
+    <origin xyz="0.2 -0.2 -0.05" rpy="1.570796  0 0"/>
   </joint>
-  <link name="wheel_front_left">
-    <inertial>
-            <mass value="2" />
-            <inertia ixx="1e-3" ixy="0.0" ixz="0"
-            iyy="1e-3" iyz="0" izz="1e-3" />
-    </inertial>
+   <link name="right_wheel_backside">
     <visual>
       <geometry>
-          <cylinder radius="0.15" length="0.1"/>
+        <cylinder radius="0.04" length="0.05" />
       </geometry>
-      <material name="white">
-        <color rgba="1 1 1 1"/>
+      <material name="red">
+        <color rgba="1 0 0 1"/>
       </material>
     </visual>
-    <collision>
-      <geometry>
-          <cylinder radius="0.15" length="0.1"/>
-      </geometry>
-      <contact_coefficients mu="1" kp="1e+13" kd="1.0"/>
-    </collision>
   </link>
-  <joint name="wheel_front_left_joint" type="continuous">
-    <origin xyz="0.25 -0.4 0.0" rpy="1.57 0.0 0.0"/>
-    <parent link="chassis"/>
-    <child link="wheel_front_left"/>
-    <axis xyz="0.0 0.0 1.0"/>
-  </joint>
-<link name="wheel_back_right">
-    <inertial>
-            <mass value="2" />
-            <inertia ixx="1e-3" ixy="0.0" ixz="0"
-            iyy="1e-3" iyz="0" izz="1e-3" />
-    </inertial>
-    <visual>
-      <geometry>
-          <cylinder radius="0.15" length="0.1"/>
-      </geometry>
-      <material name="white">
-        <color rgba="1 1 1 1"/>
-      </material>
-    </visual>
-    <collision>
-      <geometry>
-          <cylinder radius="0.15" length="0.1"/>
-      </geometry>
-      <contact_coefficients mu="1" kp="1e+13" kd="1.0"/>
-    </collision>
-  </link>
-  <joint name="wheel_back_right_joint" type="continuous">
-    <origin xyz="-0.25 0.4 0.0" rpy="1.57 0.0 0.0"/>
-    <parent link="chassis"/>
-    <child link="wheel_back_right"/>
-    <axis xyz="0.0 0.0 1.0"/>
-  </joint>
-  <link name="wheel_back_left">
-    <inertial>
-            <mass value="2" />
-            <inertia ixx="1e-3" ixy="0.0" ixz="0"
-            iyy="1e-3" iyz="0" izz="1e-3" />
-    </inertial>
-    <visual>
-      <geometry>
-          <cylinder radius="0.15" length="0.1"/>
-      </geometry>
-      <material name="white">
-        <color rgba="1 1 1 1"/>
-      </material>
-    </visual>
-    <collision>
-      <geometry>
-          <cylinder radius="0.15" length="0.1"/>
-      </geometry>
-      <contact_coefficients mu="1" kp="1e+13" kd="1.0"/>
-    </collision>
-  </link>
-  <joint name="wheel_back_left_joint" type="continuous">
-    <origin xyz="-0.25 -0.4 0.0" rpy="1.57 0.0 0.0"/>
-    <parent link="chassis"/>
-    <child link="wheel_back_left"/>
-    <axis xyz="0.0 0.0 1.0"/>
-  </joint>
-  <link name="camera">
-    <inertial>
-            <mass value="0.5" />
-            <inertia ixx="0.01" ixy="0.0" ixz="0"
-            iyy="0.01" iyz="0" izz="0.01" />
-    </inertial>
-    <visual>
-      <geometry>
-        <box size="0.1 0.5 0.2"/>
-      </geometry>
-      <material name="blue">
-        <color rgba="0 0 1 1"/>
-      </material>
-    </visual>
-    <collision>
-      <geometry>
-          <box size="0.1 0.5 0.2"/>
-      </geometry>
-    </collision>
-  </link>
-  <joint name="camera_joint" type="fixed">
-    <origin xyz="-0.35 0 0.15" rpy="0 0.0 3.14"/>
-    <parent link="chassis"/>
-    <child link="camera"/>
-    <axis xyz="0.0 0.0 1.0"/>
-  </joint>
-  <link name="lidar">
-    <inertial>
-            <mass value="0.5" />
-            <inertia ixx="0.01" ixy="0.0" ixz="0"
-            iyy="0.01" iyz="0" izz="0.01" />
-    </inertial>
-    <visual>
-      <geometry>
-        <cylinder radius="0.1" length="0.1"/>
-      </geometry>
-      <material name="red">
-        <color rgba="1 0 0  1"/>
-      </material>
-    </visual>
-    <collision>
-      <geometry>
-        <cylinder radius="0.1" length="0.1"/>
-      </geometry>
-    </collision>
-  </link>
-  <joint name="lidar_joint" type="fixed">
-    <origin xyz="-0.43 0 0.0" rpy="0 0.0 1.57"/>
-    <parent link="chassis"/>
-    <child link="lidar"/>
-    <axis xyz="0.0 0.0 1.0"/>
-  </joint>
-<!-- DIFFENERNTIAL DRIVEEEEEEEEEEEEE -->
-  <gazebo>
-<plugin name='diff_drive' filename='libgazebo_ros_diff_drive.so'>
-        <left_joint>wheel_front_left_joint</left_joint>
-        <right_joint>wheel_front_right_joint</right_joint>
-        <wheel_separation>0.8</wheel_separation>
-        <wheel_diameter>0.3</wheel_diameter>
-        <max_wheel_torque>20</max_wheel_torque>
-        <max_wheel_acceleration>1.0</max_wheel_acceleration>]
-        <publish_odom>true</publish_odom>
-        <publish_odom_tf>true</publish_odom_tf>
-        <publish_wheel_tf>true</publish_wheel_tf>
-        <odometry_frame>base_footprint</odometry_frame>
-        <robot_base_frame>chassis</robot_base_frame>
-      </plugin>
-</gazebo>
-<!-- CAMERAAAAAAAAAAAAAAAAAAAAAAAAAAAAAA -->
-      <gazebo reference="camera">
-    <sensor type="camera" name="camera1">
-      <update_rate>30.0</update_rate>
-      <camera name="head">
-        <horizontal_fov>1.3962634</horizontal_fov>
-        <image>
-          <width>800</width>
-          <height>800</height>
-          <format>R8G8B8</format>
-        </image>
-        <clip>
-          <near>0.02</near>
-          <far>300</far>
-        </clip>
-        <noise>
-          <type>gaussian</type>
-          <mean>0.0</mean>
-          <stddev>0.007</stddev>
-        </noise>
-      </camera>
-      <plugin name="camera_controller" filename="libgazebo_ros_camera.so">
-        <alwaysOn>true</alwaysOn>
-        <updateRate>0.0</updateRate>
-        <cameraName>/camera</cameraName>
-        <imageTopicName>image_raw</imageTopicName>
-        <cameraInfoTopicName>camera_info</cameraInfoTopicName>
-        <frameName>camera_link</frameName>
-        <hackBaseline>0.07</hackBaseline>
-      </plugin>
-    </sensor>
-    <material>Gazebo/Blue</material>
-  </gazebo>
-<!-- LIDAAAAAAAAAAAAAAAAAAAAAAAAAAR -->
-   <gazebo reference="lidar">
-    <sensor name="gazebo_lidar" type="ray">
-      <visualize>true</visualize>
-      <update_rate>12.0</update_rate>
-      <plugin filename="libgazebo_ros_ray_sensor.so" name="gazebo_lidar">
-      <ros>
-        <remapping>~/out:=scan</remapping>
-      </ros>
-      <output_type>sensor_msgs/LaserScan</output_type>
-      <frame_name>lidar</frame_name>
-      </plugin>
-      <ray>
-        <scan>
-          <horizontal>
-            <samples>360</samples>
-            <resolution>1</resolution>
-            <min_angle>0.00</min_angle>
-            <max_angle>3.14</max_angle>
-          </horizontal>
-        </scan>
-        <range>
-          <min>0.120</min>
-          <max>3.5</max>
-          <resolution>0.015</resolution>
-        </range>
-        <noise>
-          <type>gaussian</type>
-          <mean>0.0</mean>
-          <stddev>0.01</stddev>
-        </noise>
-      </ray>
-    </sensor>
-    <material>Gazebo/DarkGrey</material>
-  </gazebo>
 </robot>

File: install/description/share/description/urdf/armybot_gazebo.xacro (robot description, xacro)
@@ -1,6 +1,6 @@
 <?xml version="1.0"?>
-<robot name="rover" xmlns:xacro="http://ros.org/wiki/xacro">
+<robot name="robot" xmlns:xacro="http://ros.org/wiki/xacro">
   <!-- Wheels -->
-  <gazebo reference="wheel_front_right">
+  <gazebo reference="front_left_motor_link_to_front_left_wheel_link_joint">
     <mu1>1000000000000000.0</mu1>
     <mu2>1000000000000000.0</mu2>
@@ -11,5 +11,5 @@
     <fdir1>1 0 0</fdir1>
   </gazebo>
-  <gazebo reference="wheel_back_right">
+  <gazebo reference="front_right_motor_link_to_front_right_wheel_link_joint">
     <mu1>1000000000000000.0</mu1>
     <mu2>1000000000000000.0</mu2>
@@ -20,5 +20,5 @@
     <fdir1>1 0 0</fdir1>
   </gazebo>
-  <gazebo reference="wheel_front_left">
+ <gazebo reference="back_left_motor_link_to_back_left_wheel_link_joint">
     <mu1>1000000000000000.0</mu1>
     <mu2>1000000000000000.0</mu2>
@@ -29,5 +29,5 @@
     <fdir1>1 0 0</fdir1>
   </gazebo>
-  <gazebo reference="wheel_back_left">
+   <gazebo reference="back_right_motor_link_to_back_right_wheel_link_joint">
     <mu1>1000000000000000.0</mu1>
     <mu2>1000000000000000.0</mu2>
@@ -38,3 +38,94 @@
     <fdir1>1 0 0</fdir1>
   </gazebo>
+  <gazebo>
+      <plugin filename="ign_ros2_control-system" name="ign_ros2_control::IgnitionROS2ControlPlugin">
+        <parameters>
+          $(find bot_controller)/config/armybot_controller.yaml
+        </parameters>
+      </plugin>
+      <plugin filename="ignition-gazebo-imu-system" name="ignition::gazebo::systems::Imu">
+      </plugin>
+      <plugin filename="ignition-gazebo-sensors-system" name="ignition::gazebo::systems::Sensors">
+        <render_engine>ogre2</render_engine>
+      </plugin>
+  </gazebo>
+<!--   <gazebo reference="imu_link">
+    <sensor name="imu" type="imu">
+        <always_on>true</always_on>
+        <update_rate>100</update_rate>
+        <gz_frame_id>imu_link</gz_frame_id>
+        <topic>imu</topic>
+        <imu>
+          <angular_velocity>
+            <x>
+              <noise type="gaussian">
+                <mean>0.0</mean>
+                <stddev>2e-4</stddev>
+              </noise>
+            </x>
+            <y>
+              <noise type="gaussian">
+                <mean>0.0</mean>
+                <stddev>2e-4</stddev>
+              </noise>
+            </y>
+            <z>
+              <noise type="gaussian">
+                <mean>0.0</mean>
+                <stddev>2e-4</stddev>
+              </noise>
+            </z>
+          </angular_velocity>
+          <linear_acceleration>
+            <x>
+              <noise type="gaussian">
+                <mean>0.0</mean>
+                <stddev>1.7e-2</stddev>
+              </noise>
+            </x>
+            <y>
+              <noise type="gaussian">
+                <mean>0.0</mean>
+                <stddev>1.7e-2</stddev>
+              </noise>
+            </y>
+            <z>
+              <noise type="gaussian">
+                <mean>0.0</mean>
+                <stddev>1.7e-2</stddev>
+              </noise>
+            </z>
+          </linear_acceleration>
+        </imu>
+    </sensor>
+  </gazebo>-->
+  <gazebo reference="lidar_link">
+    <sensor name="lidar" type="ray">
+      <always_on>true</always_on>
+      <visualize>true</visualize>
+      <topic>scan</topic>
+      <update_rate>5</update_rate>
+      <gz_frame_id>laser_link</gz_frame_id>
+      <ray>
+        <scan>
+          <horizontal>
+            <samples>360</samples>
+            <resolution>1.00000</resolution>
+            <min_angle>0.000000</min_angle>
+            <max_angle>6.280000</max_angle>
+          </horizontal>
+        </scan>
+        <range>
+          <min>0.120000</min>
+          <max>12.0</max>
+          <resolution>0.02</resolution>
+        </range>
+        <noise>
+          <type>gaussian</type>
+          <mean>0.0</mean>
+          <stddev>0.01</stddev>
+        </noise>
+      </ray>
+    </sensor>
+  </gazebo>
 </robot>

File: install/description/share/description/urdf/bot_ros2_control.xacro (robot description, xacro)
@@ -4,7 +4,7 @@
         <!-- ros2_control Gazebo -->
         <!-- ROS 2 Humble -->
-            <hardware>
-                <plugin>ign_ros2_control/IgnitionSystem</plugin>
-            </hardware>
+        <hardware>
+            <plugin>ign_ros2_control/IgnitionSystem</plugin>
+        </hardware>
         <!-- ros2_control Common Interfaces -->
         <joint name="wheel_right_joint">
