Commit message: imu and lidar

File: install/description/share/description/urdf/armybot.xacro (robot description, xacro)
@@ -8,4 +8,5 @@
   <xacro:include filename="$(find description)/urdf/lidar.xacro"/>
   <xacro:include filename="$(find description)/urdf/wheel.xacro"/>
+  <xacro:include filename="$(find description)/urdf/imu.xacro"/>
   <xacro:include filename="$(find description)/urdf/armybot_gazebo.xacro" />
   <xacro:include filename="$(find description)/urdf/armybot_ros2_control.xacro" />
@@ -26,8 +27,9 @@
   <xacro:robot_motor parent="first_base_link" child="back_left_motor_link" xyz="-0.10 0.040 -0.025" rpy="0 0 0" />
   <xacro:robot_motor parent="first_base_link" child="back_right_motor_link" xyz="-0.10 -0.040 -0.025" rpy="0 0 0" />
-  <xacro:wheel parent="front_left_motor_link" child="front_left_wheel_link" xyz="0.0 0.060 -0.015" rpy="1.57 0 0" robot_type="$(arg robot_type)" />
-  <xacro:wheel parent="front_right_motor_link" child="front_right_wheel_link" xyz="0.0 -0.060 -0.015" rpy="1.57 0 0" robot_type="$(arg robot_type)" />
-  <xacro:wheel parent="back_left_motor_link" child="back_left_wheel_link" xyz="0.0 0.060 -0.015" rpy="1.57 0 0" robot_type="$(arg robot_type)" />
-  <xacro:wheel parent="back_right_motor_link" child="back_right_wheel_link" xyz="0.0 -0.060 -0.015" rpy="1.57 0 0" robot_type="$(arg robot_type)" />
+  <xacro:wheel parent="front_left_motor_link" child="front_left_wheel_link" xyz="0.0 0.060 -0.015" rpy="1.57 0 0" />
+  <xacro:wheel parent="front_right_motor_link" child="front_right_wheel_link" xyz="0.0 -0.060 -0.015" rpy="1.57 0 0"  />
+  <xacro:wheel parent="back_left_motor_link" child="back_left_wheel_link" xyz="0.0 0.060 -0.015" rpy="1.57 0 0"  />
+  <xacro:wheel parent="back_right_motor_link" child="back_right_wheel_link" xyz="0.0 -0.060 -0.015" rpy="1.57 0 0"  />
   <xacro:lidar parent="third_base_link" child="lidar_link" xyz="0.04 0.0 0.035" rpy="0 0 0" />
+  <xacro:imu parent="third_base_link" child="imu_link" xyz="0.08 0.0 0.035" rpy="0 0 0" />
 </robot>

File: install/description/share/description/urdf/armybot_gazebo.xacro (robot description, xacro)
@@ -50,5 +50,5 @@
       </plugin>
   </gazebo>
-<!--   <gazebo reference="imu_link">
+   <gazebo reference="imu_link">
     <sensor name="imu" type="imu">
         <always_on>true</always_on>
@@ -99,12 +99,12 @@
         </imu>
     </sensor>
-  </gazebo>-->
+  </gazebo>
   <gazebo reference="lidar_link">
-    <sensor name="lidar" type="ray">
+    <sensor name="lidar" type="gpu_ray">
       <always_on>true</always_on>
       <visualize>true</visualize>
       <topic>scan</topic>
       <update_rate>5</update_rate>
-      <gz_frame_id>laser_link</gz_frame_id>
+      <gz_frame_id>lidar_link</gz_frame_id>
       <ray>
         <scan>

File: install/description/share/description/urdf/lidar.xacro (robot description, xacro)
@@ -5,5 +5,5 @@
       <visual>
         <geometry>
-          <box size="0.10 0.075 0.060" />
+          <box size="0.05 0.045 0.040" />
         </geometry>
         <material name="red">
@@ -13,5 +13,5 @@
       <collision>
         <geometry>
-          <box size="0.10 0.075 0.060" />
+          <box size="0.05 0.045 0.040" />
         </geometry>
       </collision>

File: install/description/share/description/urdf/wheel.xacro (robot description, xacro)
@@ -1,5 +1,5 @@
 <?xml version="1.0"?>
 <robot xmlns:xacro="http://wiki.ros.org/xacro">
-  <xacro:macro name="wheel" params="parent child xyz rpy robot_type">
+  <xacro:macro name="wheel" params="parent child xyz rpy">
     <link name="${child}">
       <visual>
@@ -21,20 +21,10 @@
       </inertial>
     </link>
-    <xacro:if value="${robot_type == 'omni'}">
-      <joint name="${parent}_to_${child}_joint" type="fixed">
+    <joint name="${parent}_to_${child}_joint" type="continuous">
         <axis xyz="0.0 0.0 1"/>
         <origin xyz="${xyz}" rpy="${rpy}" />
         <parent link="${parent}" />
         <child link="${child}" />
-      </joint>
-    </xacro:if>
-    <xacro:if value="${robot_type == 'diff'}">
-      <joint name="${parent}_to_${child}_joint" type="continuous">
-        <axis xyz="0.0 0.0 1"/>
-        <origin xyz="${xyz}" rpy="${rpy}" />
-        <parent link="${parent}" />
-        <child link="${child}" />
-      </joint>
-    </xacro:if>
+    </joint>
   </xacro:macro>
 </robot>
